File: pico-th-epaper-display/pcb/pico-epaper-th.kicad_pcb (KiCad board)
At the start: 2 copper layers, 6 parts, among them Q1 AO3407, U2 TPL5110, U3 WS_1_54_epaper_module

Commit message: updated pcb design
Parts:
- added C1: 10u, Capacitor_SMD:C_0603_1608Metric_Pad1.08x0.95mm_HandSolder, F.Cu at (149.2, 78.0)
- added C2: 100n, Capacitor_SMD:C_0603_1608Metric_Pad1.08x0.95mm_HandSolder, F.Cu at (159.5, 80.3)
- added C3: 100n, Capacitor_SMD:C_0603_1608Metric_Pad1.08x0.95mm_HandSolder, F.Cu at (149.7, 85.5)
- added REF**: MountingHole_2.2mm_M2_Pad, MountingHole:MountingHole_2.2mm_M2_Pad, F.Cu at (160.9, 132.8)
- added REF**: MountingHole_2.2mm_M2_Pad, MountingHole:MountingHole_2.2mm_M2_Pad, F.Cu at (117.3, 120.1)
- added REF**: MountingHole_2.2mm_M2_Pad, MountingHole:MountingHole_2.2mm_M2_Pad, F.Cu at (117.3, 92.1)
- added REF**: MountingHole_2.2mm_M2_Pad, MountingHole:MountingHole_2.2mm_M2_Pad, F.Cu at (160.3, 92.1)
- added REF**: MountingHole_2.2mm_M2_Pad, MountingHole:MountingHole_2.2mm_M2_Pad, F.Cu at (108.9, 80.3)
- added REF**: MountingHole_2.2mm_M2_Pad, MountingHole:MountingHole_2.2mm_M2_Pad, F.Cu at (160.3, 120.1)
- added U1: GY-SHT31-D, Connector_PinHeader_2.54mm:PinHeader_1x04_P2.54mm_Vertical, F.Cu at (116.5, 136.6)
- R1: footprint Resistor_SMD:R_0201_0603Metric_Pad0.64x0.40mm_HandSolder -> Resistor_SMD:R_0603_1608Metric_Pad0.98x0.95mm_HandSolder
- moved A1 73.0 mm to (135.6, 99.6), turned to 0 degrees
- moved Q1 71.2 mm to (154.5, 76.1)
- moved U2 63.8 mm to (159.3, 85.3)
- moved R1 56.2 mm to (154.9, 83.4), turned to 90 degrees
- moved BT1 55.7 mm to (166.4, 94.3)
- moved U3 49.3 mm to (104.4, 114.1), turned to 180 degrees
Other:
- board outline added: 70 x 70 mm
- board text added: "1.54inch e-paper"

Commit message: updated pcb
Connections:
- A1 pad 20: Net-(A1-GPIO15) -> unconnected-(A1-GPIO15-Pad20)
- A1 pad 34: unconnected-(A1-GPIO28_ADC2-Pad34) -> Net-(A1-GPIO28_ADC2)
- U2 pad 4: Net-(A1-GPIO15) -> Net-(A1-GPIO28_ADC2)
Changed lines of the file:
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@@
 			(layers "F.Cu" "F.Mask" "F.Paste")
 			(roundrect_rratio 0.25)
-			(net "Net-(A1-GPIO15)")
+			(net "Net-(A1-GPIO28_ADC2)")
 			(pinfunction "DONE_4")
 			(pintype "input")
@@
 			(layers "F.Cu" "F.Mask")
 			(roundrect_rratio 0.5)
-			(net "Net-(A1-GPIO15)")
+			(net "unconnected-(A1-GPIO15-Pad20)")
 			(pinfunction "GPIO15_20")
-			(pintype "bidirectional")
+			(pintype "bidirectional+no_connect")
 		)
 		(pad "21" smd roundrect
@@
 			(layers "F.Cu" "F.Mask")
 			(roundrect_rratio 0.5)
-			(net "unconnected-(A1-GPIO28_ADC2-Pad34)")
+			(net "Net-(A1-GPIO28_ADC2)")
 			(pinfunction "GPIO28_ADC2_34")
-			(pintype "bidirectional+no_connect")
+			(pintype "bidirectional")
 		)
 		(pad "35" smd roundrect

Commit message: pcb updated
Parts:
- U3: footprint Connector_PinHeader_2.54mm:PinHeader_1x09_P2.54mm_Vertical -> Connector_PinHeader_2.54mm:PinHeader_1x08_P2.54mm_Vertical
- moved C2 5.82 mm to (155.4, 84.4), turned to 180 degrees
- moved REF** 4.53 mm to (160.4, 137.3)
- moved R1 3.60 mm to (151.9, 81.4)
- moved U3 3.43 mm to (107.1, 116.2)
- moved REF** 3.35 mm to (110.4, 77.3)
- moved REF** 1.71 mm to (160.1, 93.8)
- moved REF** 1.71 mm to (160.1, 121.8)
- moved REF** 1.71 mm to (117.1, 121.8)
- moved REF** 1.71 mm to (117.1, 93.8)
- moved BT1 1.22 mm to (166.2, 93.1)
- moved Q1 0.87 mm to (153.9, 75.5)
- moved U1 0.78 mm to (116.2, 135.9)
- moved C3 0.73 mm to (148.9, 85.6)
- moved C1 0.27 mm to (148.9, 77.9)
- moved A1 0.26 mm to (135.4, 99.5)
Other:
- outline, holes or cut-outs redrawn
