File: pico-th-epaper-display/pcb/pico-epaper-th.kicad_sch (KiCad schematic)
At the start: 7 parts, among them Q1 AO3407, U1 GY-SHT31-D, U2 TPL5110, U3 WS_1_54_epaper_module

Commit message: updated pcb design
Parts:
- added C1: 10u, Capacitor_SMD:C_0603_1608Metric_Pad1.08x0.95mm_HandSolder, symbol Device:C
- added C2, C3: 100n, Capacitor_SMD:C_0603_1608Metric_Pad1.08x0.95mm_HandSolder, symbol Device:C
- R1: footprint Resistor_SMD:R_0201_0603Metric_Pad0.64x0.40mm_HandSolder -> Resistor_SMD:R_0603_1608Metric_Pad0.98x0.95mm_HandSolder
- U1: footprint (none) -> Connector_PinHeader_2.54mm:PinHeader_1x04_P2.54mm_Vertical
Connections:
- net GND: now also C1.2, C2.2, C3.2
- net VCC: now also C2.1
- net at A1.36 (3V3), U1.1 (VCC), U3.8 (VCC): now also C3.1
- net at A1.39 (VSYS), Q1.3 (D): now also C1.1

Commit message: updated pcb
Connections:
- net at U2.4 (DONE): now also A1.34 (GPIO28_ADC2); no longer A1.20 (GPIO15)
Changed lines of the file:
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@@
+	)
+	(no_connect
+		(at 80.01 86.36)
+	)
+	(no_connect
+		(at 125.73 109.22)
+	)
+	(no_connect
+		(at 80.01 66.04)
+	)
+	(no_connect
+		(at 125.73 91.44)
+	)
+	(no_connect
+		(at 125.73 104.14)
+	)
+	(no_connect
+		(at 125.73 83.82)
+	)
+	(no_connect
+		(at 80.01 81.28)
+	)
+	(no_connect
+		(at 80.01 76.2)
+	)
+	(no_connect
+		(at 80.01 96.52)
 	)
 	(no_connect
@@
 	)
 	(no_connect
-		(at 80.01 86.36)
-	)
-	(no_connect
-		(at 125.73 109.22)
-	)
-	(no_connect
-		(at 80.01 66.04)
-	)
-	(no_connect
-		(at 125.73 91.44)
-	)
-	(no_connect
-		(at 125.73 104.14)
-	)
-	(no_connect
-		(at 125.73 83.82)
-	)
-	(no_connect
-		(at 80.01 81.28)
-	)
-	(no_connect
-		(at 80.01 76.2)
-	)
-	(no_connect
-		(at 80.01 96.52)
-	)
-	(no_connect
 		(at 80.01 99.06)
 	)
@@
 	)
 	(no_connect
+		(at 80.01 119.38)
+	)
+	(no_connect
 		(at 102.87 58.42)
 	)
@@
 	)
 	(no_connect
-		(at 125.73 114.3)
-	)
-	(no_connect
 		(at 80.01 88.9)
 	)
@@
 	(wire
 		(pts
+			(xy 143.51 93.98) (xy 143.51 114.3)
+		)
+		(stroke
+			(width 0)
+			(type default)
+		)
+	)
+	(wire
+		(pts
 			(xy 176.53 76.2) (xy 203.2 76.2)
 		)
@@
 	(wire
 		(pts
-			(xy 143.51 137.16) (xy 68.58 137.16)
-		)
-		(stroke
-			(width 0)
-			(type default)
-		)
-	)
-	(wire
-		(pts
 			(xy 132.08 76.2) (xy 138.43 76.2)
 		)
@@
 	(wire
 		(pts
-			(xy 68.58 119.38) (xy 80.01 119.38)
-		)
-		(stroke
-			(width 0)
-			(type default)
-		)
-	)
-	(wire
-		(pts
 			(xy 53.34 111.76) (xy 58.42 111.76)
 		)
@@
 	(wire
 		(pts
+			(xy 143.51 114.3) (xy 125.73 114.3)
+		)
+		(stroke
+			(width 0)
+			(type default)
+		)
+	)
+	(wire
+		(pts
 			(xy 203.2 105.41) (xy 203.2 110.49)
 		)
@@
 	(wire
 		(pts
+			(xy 62.23 53.34) (xy 74.93 53.34)
+		)
+		(stroke
+			(width 0)
+			(type default)
+		)
+	)
+	(wire
+		(pts
+			(xy 71.12 99.06) (xy 71.12 111.76)
+		)
+		(stroke
+			(width 0)
+			(type default)
+		)
+	)
+	(wire
+		(pts
+			(xy 176.53 104.14) (xy 176.53 110.49)
+		)
+		(stroke
+			(width 0)
+			(type default)
+		)
+	)
+	(wire
+		(pts
+			(xy 55.88 58.42) (xy 55.88 53.34)
+		)
+		(stroke
+			(width 0)
+			(type default)
+		)
+	)
+	(wire
+		(pts
+			(xy 127 57.15) (xy 127 58.42)
+		)
+		(stroke
+			(width 0)
+			(type default)
+		)
+	)
+	(wire
+		(pts
+			(xy 107.95 53.34) (xy 107.95 58.42)
+		)
+		(stroke
+			(width 0)
+			(type default)
+		)
+	)
+	(wire
+		(pts
+			(xy 132.08 46.99) (xy 132.08 76.2)
+		)
+		(stroke
+			(width 0)
+			(type default)
+		)
+	)
+	(wire
+		(pts
+			(xy 58.42 111.76) (xy 58.42 123.19)
+		)
+		(stroke
+			(width 0)
+			(type default)
+		)
+	)
+	(wire
+		(pts
 			(xy 163.83 93.98) (xy 143.51 93.98)
 		)
@@
 	(wire
 		(pts
-			(xy 62.23 53.34) (xy 74.93 53.34)
-		)
-		(stroke
-			(width 0)
-			(type default)
-		)
-	)
-	(wire
-		(pts
-			(xy 71.12 99.06) (xy 71.12 111.76)
-		)
-		(stroke
-			(width 0)
-			(type default)
-		)
-	)
-	(wire
-		(pts
-			(xy 176.53 104.14) (xy 176.53 110.49)
-		)
-		(stroke
-			(width 0)
-			(type default)
-		)
-	)
-	(wire
-		(pts
-			(xy 55.88 58.42) (xy 55.88 53.34)
-		)
-		(stroke
-			(width 0)
-			(type default)
-		)
-	)
-	(wire
-		(pts
-			(xy 127 57.15) (xy 127 58.42)
-		)
-		(stroke
-			(width 0)
-			(type default)
-		)
-	)
-	(wire
-		(pts
-			(xy 107.95 53.34) (xy 107.95 58.42)
-		)
-		(stroke
-			(width 0)
-			(type default)
-		)
-	)
-	(wire
-		(pts
-			(xy 132.08 46.99) (xy 132.08 76.2)
-		)
-		(stroke
-			(width 0)
-			(type default)
-		)
-	)
-	(wire
-		(pts
-			(xy 143.51 93.98) (xy 143.51 137.16)
-		)
-		(stroke
-			(width 0)
-			(type default)
-		)
-	)
-	(wire
-		(pts
-			(xy 58.42 111.76) (xy 58.42 123.19)
-		)
-		(stroke
-			(width 0)
-			(type default)
-		)
-	)
-	(wire
-		(pts
 			(xy 53.34 109.22) (xy 80.01 109.22)
 		)
@@
 		)
 		(stroke
-			(width 0)
-			(type default)
-		)
-	)
-	(wire
-		(pts
-			(xy 68.58 137.16) (xy 68.58 119.38)
-		)
-		(stroke

Commit message: pcb updated
Parts:
- U3: footprint Connector_PinHeader_2.54mm:PinHeader_1x09_P2.54mm_Vertical -> Connector_PinHeader_2.54mm:PinHeader_1x08_P2.54mm_Vertical
Changed lines of the file:
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@@
 			)
 		)
-		(property "Footprint" "Connector_PinHeader_2.54mm:PinHeader_1x09_P2.54mm_Vertical"
+		(property "Footprint" "Connector_PinHeader_2.54mm:PinHeader_1x08_P2.54mm_Vertical"
 			(at 44.45 89.916 0)
 			(hide yes)
