File: 001-pico-th-epaper-display/pcb/pico-epaper-th.kicad_pcb (KiCad board)
At the start: 2 copper layers, 70 x 70 mm, 17 parts, among them Q1 AO3407, U1 GY-SHT31-D, U2 TPL5110, U3 WS_1_54_epaper_module

Commit message: pcb routing
Routing:
- net /3V3: track 3.26 -> 97.6 mm, vias 0 -> 1
Changed lines of the file:
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@@
+	)
+	(segment
+		(start 145.06 85.5)
+		(end 145.09 85.53)
+		(width 0.8)
+		(layer "F.Cu")
+		(net "/3V3")
 	)
 	(segment
@@
 		(net "/3V3")
 	)
+	(segment
+		(start 138.2 85.5)
+		(end 145.06 85.5)
+		(width 0.8)
+		(layer "F.Cu")
+		(net "/3V3")
+	)
+	(via
+		(at 138.2 85.5)
+		(size 0.8)
+		(drill 0.4)
+		(layers "F.Cu" "B.Cu")
+		(net "/3V3")
+	)
+	(segment
+		(start 127.55 98.45)
+		(end 136.8 89.2)
+		(width 0.8)
+		(layer "B.Cu")
+		(net "/3V3")
+	)
+	(segment
+		(start 136.8 86.9)
+		(end 138.2 85.5)
+		(width 0.8)
+		(layer "B.Cu")
+		(net "/3V3")
+	)
+	(segment
+		(start 107.1 98.45)
+		(end 127.55 98.45)
+		(width 0.8)
+		(layer "B.Cu")
+		(net "/3V3")
+	)
+	(segment
+		(start 136.8 89.2)
+		(end 136.8 86.9)
+		(width 0.8)
+		(layer "B.Cu")
+		(net "/3V3")
+	)
+	(segment
+		(start 154.7 136.88)
+		(end 127.55 109.73)
+		(width 0.8)
+		(layer "B.Cu")
+		(net "/3V3")
+	)
+	(segment
+		(start 127.55 109.73)
+		(end 127.55 98.45)
+		(width 0.8)
+		(layer "B.Cu")
+		(net "/3V3")
+	)

Commit message: pcb routing
Routing:
- net /3V3: track 97.6 -> 130.6 mm
Changed lines of the file:
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@@
+	)
+	(segment
+		(start 133.32 136.88)
+		(end 154.7 136.88)
+		(width 0.8)
+		(layer "F.Cu")
+		(net "/3V3")
 	)
 	(segment
@@
 	)
 	(segment
+		(start 138.2 85.5)
+		(end 130 93.7)
+		(width 0.8)
+		(layer "F.Cu")
+		(net "/3V3")
+	)
+	(segment
+		(start 130 93.7)
+		(end 130 133.6)
+		(width 0.8)
+		(layer "F.Cu")
+		(net "/3V3")
+	)
+	(segment
+		(start 133.3 136.9)
+		(end 133.32 136.88)
+		(width 0.8)
+		(layer "F.Cu")
+		(net "/3V3")
+	)
+	(segment
 		(start 145.06 85.5)
 		(end 145.09 85.53)
@@
 		(start 148.3075 85.53)
 		(end 148.3375 85.5)
+		(width 0.8)
+		(layer "F.Cu")
+		(net "/3V3")
+	)
+	(segment
+		(start 130 133.6)
+		(end 133.3 136.9)
 		(width 0.8)
 		(layer "F.Cu")
@@
 	)
 	(segment
-		(start 127.55 98.45)
-		(end 136.8 89.2)
-		(width 0.8)
-		(layer "B.Cu")
-		(net "/3V3")
-	)
-	(segment
-		(start 136.8 86.9)
+		(start 109.1 85.5)
 		(end 138.2 85.5)
 		(width 0.8)
@@
 	(segment
 		(start 107.1 98.45)
-		(end 127.55 98.45)
-		(width 0.8)
-		(layer "B.Cu")
-		(net "/3V3")
-	)
-	(segment
-		(start 136.8 89.2)
-		(end 136.8 86.9)
-		(width 0.8)
-		(layer "B.Cu")
-		(net "/3V3")
-	)
-	(segment
-		(start 154.7 136.88)
-		(end 127.55 109.73)
-		(width 0.8)
-		(layer "B.Cu")
-		(net "/3V3")
-	)
-	(segment
-		(start 127.55 109.73)
-		(end 127.55 98.45)
+		(end 107.1 87.5)
+		(width 0.8)
+		(layer "B.Cu")
+		(net "/3V3")
+	)
+	(segment
+		(start 107.1 87.5)
+		(end 109.1 85.5)
 		(width 0.8)
 		(layer "B.Cu")
@@
 		(layer "F.Cu")
 		(net "VCC")
+	)
+	(segment
+		(start 163.95 82.525)
+		(end 166.05 82.525)
+		(width 0.2)
+		(layer "F.Cu")
+		(net "Net-(U2-DELAY{slash}M_DRV)")
+	)
+	(segment
+		(start 166.05 82.525)
+		(end 166.1 82.575)
+		(width 0.2)
+		(layer "F.Cu")
+		(net "Net-(U2-DELAY{slash}M_DRV)")
 	)
 	(segment
@@
 		(net "Net-(A1-GPIO20)")
 	)
-	(segment
-		(start 163.95 82.525)
-		(end 166.05 82.525)
-		(width 0.2)
-		(layer "F.Cu")
-		(net "Net-(U2-DELAY{slash}M_DRV)")
-	)
-	(segment
-		(start 166.05 82.525)
-		(end 166.1 82.575)
-		(width 0.2)
-		(layer "F.Cu")
-		(net "Net-(U2-DELAY{slash}M_DRV)")
-	)
 	(zone

Commit message: pcb updated
Routing:
- net Net-(A1-GPIO9): track 20.8 -> 43.2 mm, vias 1 -> 0
- net Net-(A1-GPIO8): track 44.4 -> 48.5 mm
- net Net-(A1-VSYS): track 8.36 -> 10.2 mm
- net Net-(A1-GPIO10): track 37.8 -> 39.4 mm
- net Net-(A1-GPIO20): track 25.4 -> 26.6 mm
- net VCC: track 25.5 -> 26.2 mm
Changed lines of the file:
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@@
-	)
-	(segment
-		(start 107.1 111.15)
-		(end 103.1 107.15)
-		(width 0.2)
-		(layer "F.Cu")
-		(net "Net-(A1-GPIO8)")
-	)
-	(segment
-		(start 103.1 107.15)
-		(end 103.1 93.9)
-		(width 0.2)
-		(layer "F.Cu")
-		(net "Net-(A1-GPIO8)")
-	)
-	(segment
-		(start 103.1 93.9)
-		(end 111.7 93.9)
-		(width 0.2)
-		(layer "F.Cu")
-		(net "Net-(A1-GPIO8)")
 	)
 	(segment
@@
 	)
 	(segment
+		(start 101.8 110.4)
+		(end 101.8 94.5)
+		(width 0.2)
+		(layer "F.Cu")
+		(net "Net-(A1-GPIO8)")
+	)
+	(segment
+		(start 107.1 111.15)
+		(end 102.55 111.15)
+		(width 0.2)
+		(layer "F.Cu")
+		(net "Net-(A1-GPIO8)")
+	)
+	(segment
 		(start 118.63 100.77)
 		(end 125.71 100.77)
@@
 	)
 	(segment
+		(start 102.4 93.9)
+		(end 111.7 93.9)
+		(width 0.2)
+		(layer "F.Cu")
+		(net "Net-(A1-GPIO8)")
+	)
+	(segment
 		(start 111.7 93.9)
 		(end 118.6 100.8)
@@
 	)
 	(segment
-		(start 121.1 103.3)
-		(end 121.4 103.3)
+		(start 101.8 94.5)
+		(end 102.4 93.9)
+		(width 0.2)
+		(layer "F.Cu")
+		(net "Net-(A1-GPIO8)")
+	)
+	(segment
+		(start 102.55 111.15)
+		(end 101.8 110.4)
+		(width 0.2)
+		(layer "F.Cu")
+		(net "Net-(A1-GPIO8)")
+	)
+	(segment
+		(start 103.1 107.9)
+		(end 103.1 95.3)
 		(width 0.2)
 		(layer "F.Cu")
@@
 	)
 	(segment
-		(start 121.41 103.31)
+		(start 110.9 94.8)
+		(end 119.41 103.31)
+		(width 0.2)
+		(layer "F.Cu")
+		(net "Net-(A1-GPIO9)")
+	)
+	(segment
+		(start 119.41 103.31)
 		(end 125.71 103.31)
 		(width 0.2)
@@
 	)
 	(segment
-		(start 121.4 103.3)
-		(end 121.41 103.31)
+		(start 103.6 94.8)
+		(end 110.9 94.8)
 		(width 0.2)
 		(layer "F.Cu")
 		(net "Net-(A1-GPIO9)")
 	)
-	(via
-		(at 121.1 103.3)
-		(size 0.6)
-		(drill 0.3)
-		(layers "F.Cu" "B.Cu")
+	(segment
+		(start 103.1 95.3)
+		(end 103.6 94.8)
+		(width 0.2)
+		(layer "F.Cu")
 		(net "Net-(A1-GPIO9)")
 	)
 	(segment
-		(start 112.41 103.3)
-		(end 121.1 103.3)
-		(width 0.2)
-		(layer "B.Cu")
+		(start 107.1 108.61)
+		(end 103.81 108.61)
+		(width 0.2)
+		(layer "F.Cu")
 		(net "Net-(A1-GPIO9)")
 	)
 	(segment
-		(start 107.1 108.61)
-		(end 112.41 103.3)
-		(width 0.2)
-		(layer "B.Cu")
+		(start 103.81 108.61)
+		(end 103.1 107.9)
+		(width 0.2)
+		(layer "F.Cu")
 		(net "Net-(A1-GPIO9)")
+	)
+	(segment
+		(start 104.7 95.7)
+		(end 109.4 95.7)
+		(width 0.2)
+		(layer "F.Cu")
+		(net "Net-(A1-GPIO10)")
+	)
+	(segment
+		(start 122.09 108.39)
+		(end 125.71 108.39)
+		(width 0.2)
+		(layer "F.Cu")
+		(net "Net-(A1-GPIO10)")
+	)
+	(segment
+		(start 104.3 96.1)
+		(end 104.7 95.7)
+		(width 0.2)
+		(layer "F.Cu")
+		(net "Net-(A1-GPIO10)")
+	)
+	(segment
+		(start 125.56 107.84)
+		(end 125.71 107.99)
+		(width 0.2)
+		(layer "F.Cu")
+		(net "Net-(A1-GPIO10)")
+	)
+	(segment
+		(start 104.3 105.4)
+		(end 104.3 96.1)
+		(width 0.2)
+		(layer "F.Cu")
+		(net "Net-(A1-GPIO10)")
+	)
+	(segment
+		(start 104.97 106.07)
+		(end 104.3 105.4)
+		(width 0.2)
+		(layer "F.Cu")
+		(net "Net-(A1-GPIO10)")
 	)
 	(segment
@@
 	(segment
 		(start 107.1 106.07)
-		(end 104.7 103.67)
-		(width 0.2)
-		(layer "F.Cu")
-		(net "Net-(A1-GPIO10)")
-	)
-	(segment
-		(start 104.7 103.67)
-		(end 104.7 95.7)
-		(width 0.2)
-		(layer "F.Cu")
-		(net "Net-(A1-GPIO10)")
-	)
-	(segment
-		(start 125.56 107.84)
-		(end 125.71 107.99)
-		(width 0.2)
-		(layer "F.Cu")
-		(net "Net-(A1-GPIO10)")
-	)
-	(segment
-		(start 104.7 95.7)
-		(end 109.4 95.7)
-		(width 0.2)
-		(layer "F.Cu")
-		(net "Net-(A1-GPIO10)")
-	)
-	(segment
-		(start 122.09 108.39)
-		(end 125.71 108.39)
+		(end 104.97 106.07)
 		(width 0.2)
 		(layer "F.Cu")
@@
 	)
 	(segment
-		(start 160.025 82.525)
-		(end 162.05 82.525)
-		(width 0.8)
-		(layer "F.Cu")
-		(net "VCC")
-	)
-	(segment
-		(start 160 79.7)
-		(end 160 82.5)
+		(start 148.3 78.2375)
+		(end 150.1 78.2375)
+		(width 0.8)
+		(layer "F.Cu")
+		(net "Net-(A1-VSYS)")
+	)
+	(segment
+		(start 158.5 83.4)
+		(end 158.5 78.2)
+		(width 0.8)
+		(layer "F.Cu")
+		(net "VCC")
+	)
+	(segment
+		(start 159.7 77.5)
+		(end 159.7 77.8)
+		(width 0.8)
+		(layer "F.Cu")
+		(net "VCC")
+	)
+	(segment
+		(start 160.9 77.8)
+		(end 161.75 78.65)
+		(width 0.8)
+		(layer "F.Cu")
+		(net "VCC")
+	)
+	(segment
+		(start 161.75 78.65)
+		(end 161 77.9)
+		(width 0.8)
+		(layer "F.Cu")
+		(net "VCC")
+	)
+	(segment
+		(start 158.2 76)
+		(end 159.7 77.5)
 		(width 0.8)
 		(layer "F.Cu")
@@
 	)
 	(segment
-		(start 162.05 77.05)
-		(end 162.05 80.25)
-		(width 0.8)
-		(layer "F.Cu")
-		(net "VCC")
-	)
-	(segment
-		(start 156.3 76)
-		(end 161 76)
-		(width 0.8)
-		(layer "F.Cu")
-		(net "VCC")
-	)
-	(segment
 		(start 162.05 82.525)
 		(end 162.05 84.3875)
@@
 	)
 	(segment
+		(start 162.1375 84.475)
+		(end 159.575 84.475)
+		(width 0.8)
+		(layer "F.Cu")
+		(net "VCC")
+	)
+	(segment
+		(start 158.2 76)
+		(end 156.3 76)
+		(width 0.8)
+		(layer "F.Cu")
+		(net "VCC")
+	)
+	(segment
 		(start 162.05 84.3875)
 		(end 162.1375 84.475)
@@
 	)
 	(segment
-		(start 160 82.5)
-		(end 160.025 82.525)
-		(width 0.8)
-		(layer "F.Cu")
-		(net "VCC")
-	)
-	(segment
-		(start 156.3 76)
-		(end 160 79.7)
+		(start 159.7 77.8)
+		(end 160.9 77.8)
+		(width 0.8)
+		(layer "F.Cu")
+		(net "VCC")
+	)
+	(segment
+		(start 162.05 78.95)
+		(end 161.75 78.65)
+		(width 0.8)
+		(layer "F.Cu")
+		(net "VCC")
+	)
+	(segment
+		(start 158.9 77.8)
+		(end 159.7 77.8)
+		(width 0.8)
+		(layer "F.Cu")
+		(net "VCC")
+	)
+	(segment
+		(start 158.5 78.2)
+		(end 158.9 77.8)
+		(width 0.8)
+		(layer "F.Cu")
+		(net "VCC")
+	)
+	(segment
+		(start 162.05 80.25)
+		(end 162.05 78.95)
 		(width 0.8)
 		(layer "F.Cu")
@@
 	)
 	(segment
-		(start 161 76)
-		(end 162.05 77.05)
+		(start 159.575 84.475)
+		(end 158.5 83.4)
 		(width 0.8)
 		(layer "F.Cu")
@@
 	)
 	(segment
-		(start 157.2 130.9)
-		(end 155.6 130.9)
+		(start 157.2 131.5)
+		(end 157.2 109.9)
 		(width 0.2)
 		(layer "F.Cu")
@@
 	)
 	(segment
-		(start 155.6 130.9)
-		(end 154.7 131.8)
+		(start 154.7 131.8)
+		(end 156.9 131.8)
 		(width 0.2)
 		(layer "F.Cu")
@@
 	(segment
 		(start 155.69 108.39)
-		(end 157.2 109.9)
+		(end 145.09 108.39)
 		(width 0.2)
 		(layer "F.Cu")
@@
 	)
 	(segment
+		(start 156.9 131.8)
+		(end 157.2 131.5)
+		(width 0.2)
+		(layer "F.Cu")
+		(net "Net-(A1-GPIO21)")
+	)
+	(segment
 		(start 157.2 109.9)
-		(end 157.2 130.9)
+		(end 155.69 108.39)
 		(width 0.2)
 		(layer "F.Cu")
@@
 	)
 	(segment
-		(start 145.09 108.39)
-		(end 155.69 108.39)
-		(width 0.2)
-		(layer "F.Cu")
-		(net "Net-(A1-GPIO21)")
-	)
-	(segment
-		(start 154.7 129.26)
-		(end 151.4 125.96)
+		(start 145.09 110.93)
+		(end 152.43 110.93)
 		(width 0.2)
 		(layer "F.Cu")
@@
 	)
 	(segment
-		(start 150.33 110.93)
-		(end 145.09 110.93)
+		(start 152.43 110.93)
+		(end 154.7 113.2)
 		(width 0.2)
 		(layer "F.Cu")
@@
 	)
 	(segment
-		(start 151.4 125.96)
-		(end 151.4 112)
-		(width 0.2)
-		(layer "F.Cu")
-		(net "Net-(A1-GPIO20)")
-	)
-	(segment
-		(start 151.4 112)
-		(end 150.33 110.93)
+		(start 154.7 113.2)
+		(end 154.7 129.26)
 		(width 0.2)
 		(layer "F.Cu")
@@
 		(hatch edge 0.5)
 		(connect_pads
-			(clearance 0.5)
+			(clearance 0.3)
 		)
 		(min_thickness 0.25)
 		(fill yes
-			(thermal_gap 0.5)
+			(thermal_gap 0.3)
 			(thermal_bridge_width 0.5)
 			(island_removal_mode 0)

Commit message: updated pcb
Parts:
- C1: value 10u -> 0.1u
- C2, C3: value 100n -> 0.1u
- C4: value 100n -> 10u
Other:
- board text added: "Low Power T/H ePaper Display"
- board text added: "electronut.in"
Changed lines of the file:
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@@
 			)
 			(rotate
-				(xyz -0 -0 -0)
+				(xyz 180 -0 -0)
 			)
 		)
@@
 			)
 		)
-		(property "Value" "100n"
+		(property "Value" "0.1u"
 			(at 0 1.43 0)
 			(layer "F.Fab")
@@
 			)
 		)
-		(property "Value" "100n"
+		(property "Value" "10u"
 			(at 0 1.43 90)
 			(layer "F.Fab")
@@
 			)
 		)
-		(property "Value" "100n"
+		(property "Value" "0.1u"
 			(at 0 1.43 0)
 			(layer "F.Fab")
@@
 			)
 		)
-		(property "Value" "10u"
+		(property "Value" "0.1u"
 			(at 0 1.43 90)
 			(layer "F.Fab")
@@
 			)
 		)
-		(model "${KIPRJMOD}/AABattery Holder.stp"
-			(offset
-				(xyz -48 -57 -10)
-			)
-			(scale
-				(xyz 1 1 1)
-			)
-			(rotate
-				(xyz -0 -180 -0)
-			)
-		)
 	)
 	(gr_rect
@@
 		)
 	)
+	(gr_text "Low Power T/H ePaper Display"
+		(at 117.4 141 0)
+		(layer "F.SilkS")
+		(effects
+			(font
+				(size 1.5 1.5)
+				(thickness 0.3)
+				(bold yes)
+			)
+			(justify left bottom)
+		)
+	)
+	(gr_text "electronut.in"
+		(at 166.2 101.6 90)
+		(layer "B.SilkS")
+		(effects
+			(font
+				(size 1.5 1.5)
+				(thickness 0.3)
+				(bold yes)
+			)
+			(justify left bottom mirror)
+		)
+	)
